File: 8x-sata-backplane/8x-sata-backplane.kicad_pcb (KiCad board)
At the start: 4 copper layers, 129.8 x 129 mm, 13 parts

Commit message: v1.0
Parts:
- removed the REF** at (143.5, 29.0)
- removed the REF** at (125.8, 144.0)
- removed the REF** at (55.0, 144.0)
- removed the REF** at (37.3, 29.0)
- added D1: LED, LED_SMD:LED_0603_1608Metric, F.Cu at (48.5, 37.1)
- added D2: LED, LED_SMD:LED_0603_1608Metric, F.Cu at (83.8, 37.1)
- added D3: LED, LED_SMD:LED_0603_1608Metric, F.Cu at (119.4, 37.1)
- added D4: LED, LED_SMD:LED_0603_1608Metric, F.Cu at (154.7, 36.6)
- added Q1: BC850, Package_TO_SOT_SMD:SOT-23, F.Cu at (43.9, 35.8)
- added Q2: BC850, Package_TO_SOT_SMD:SOT-23, F.Cu at (79.2, 35.8)
- added Q3: BC850, Package_TO_SOT_SMD:SOT-23, F.Cu at (114.8, 35.8)
- added Q4: BC850, Package_TO_SOT_SMD:SOT-23, F.Cu at (150.1, 35.8)
- added R1: 1k, Resistor_SMD:R_0805_2012Metric, F.Cu at (40.4, 37.1)
- added R10: 1k, Resistor_SMD:R_0805_2012Metric, F.Cu at (146.6, 37.1)
- added R11: 330, Resistor_SMD:R_0805_2012Metric, F.Cu at (146.6, 35.1)
- added R12: 1k, Resistor_SMD:R_0805_2012Metric, F.Cu at (150.1, 38.9)
- added R2: 330, Resistor_SMD:R_0805_2012Metric, F.Cu at (40.4, 35.1)
- added R3: 1k, Resistor_SMD:R_0805_2012Metric, F.Cu at (43.9, 38.9)
- added R4: 1k, Resistor_SMD:R_0805_2012Metric, F.Cu at (75.7, 37.1)
- added R5: 330, Resistor_SMD:R_0805_2012Metric, F.Cu at (75.7, 35.1)
- added R6: 1k, Resistor_SMD:R_0805_2012Metric, F.Cu at (79.2, 38.9)
- added R7: 1k, Resistor_SMD:R_0805_2012Metric, F.Cu at (111.3, 37.1)
- added R8: 330, Resistor_SMD:R_0805_2012Metric, F.Cu at (111.3, 35.1)
- added R9: 1k, Resistor_SMD:R_0805_2012Metric, F.Cu at (114.8, 38.9)
- added REF**: MountingHole_3.2mm_M3, MountingHole:MountingHole_3.2mm_M3, F.Cu at (125.8, 144.0)
- added REF**: MountingHole_3.2mm_M3, MountingHole:MountingHole_3.2mm_M3, F.Cu at (143.5, 28.0)
- added REF**: MountingHole_3.2mm_M3, MountingHole:MountingHole_3.2mm_M3, F.Cu at (55.0, 144.0)
- added REF**: MountingHole_3.2mm_M3, MountingHole:MountingHole_3.2mm_M3, F.Cu at (37.3, 28.0)
- J1, J3, J5, J7: footprint shirnschall:SATA BACKPLANE RECPT VERTICAL SMT -> shirnschall:sata-backplane-connector-vert
- moved J1 1.78 mm to (44.4, 62.9)
- moved J3 1.78 mm to (79.8, 62.9)
- moved J5 1.78 mm to (115.2, 62.9)
- moved J7 1.78 mm to (150.6, 62.9)
Connections:
- J1 pad 1: /GND1 -> GND1
- J1 pad 18: GND -> 1_ACT
- J1 pad 23: unconnected-(J1-C1-Pad23) -> GND1
- J1 pad 4: /GND1 -> GND1
- J1 pad 7: /GND1 -> GND1
- J2 pad 1: /GND1 -> GND1
- J2 pad 4: /GND1 -> GND1
- J2 pad 7: /GND1 -> GND1
- J2 pad 8: unconnected-(J2-C1-Pad8) -> GND1
- J2 pad 9: unconnected-(J2-C2-Pad9) -> GND1
- J3 pad 1: /GND2 -> GND2
- J3 pad 18: GND -> 2_ACT
- J3 pad 23: unconnected-(J3-C1-Pad23) -> GND2
- J3 pad 4: /GND2 -> GND2
- J3 pad 7: /GND2 -> GND2
- J4 pad 1: /GND2 -> GND2
- J4 pad 4: /GND2 -> GND2
- J4 pad 7: /GND2 -> GND2
- J4 pad 8: unconnected-(J4-C1-Pad8) -> GND2
- J4 pad 9: unconnected-(J4-C2-Pad9) -> GND2
- J5 pad 1: /GND3 -> GND3
- J5 pad 18: GND -> 3_ACT
- J5 pad 23: unconnected-(J5-C1-Pad23) -> GND3
- J5 pad 4: /GND3 -> GND3
- J5 pad 7: /GND3 -> GND3
- J6 pad 1: /GND3 -> GND3
- J6 pad 4: /GND3 -> GND3
- J6 pad 7: /GND3 -> GND3
- J6 pad 8: unconnected-(J6-C1-Pad8) -> GND3
- J6 pad 9: unconnected-(J6-C2-Pad9) -> GND3
- J7 pad 1: /GND4 -> GND4
- J7 pad 18: GND -> 4_ACT
- J7 pad 23: unconnected-(J7-C1-Pad23) -> GND4
- J7 pad 4: /GND4 -> GND4
- J7 pad 7: /GND4 -> GND4
- J8 pad 1: /GND4 -> GND4
- J8 pad 4: /GND4 -> GND4
- J8 pad 7: /GND4 -> GND4
- J8 pad 8: unconnected-(J8-C1-Pad8) -> GND4
- J8 pad 9: unconnected-(J8-C2-Pad9) -> GND4
Routing:
- net 1_ACT: track 0.00 -> 25.1 mm
- net 3_ACT: track 0.00 -> 25.0 mm
- net 2_ACT: track 0.00 -> 24.6 mm
- net 4_ACT: track 0.00 -> 24.6 mm
- net GND4: track 0.00 -> 13.6 mm, vias 0 -> 7
- net GND1: track 0.00 -> 13.6 mm, vias 0 -> 7
- net GND3: track 0.00 -> 13.3 mm, vias 0 -> 7
- net GND: track 99.4 -> 86.3 mm, vias 48 -> 44
- net GND2: track 0.00 -> 13.1 mm, vias 0 -> 7
- net /GND4: track 11.9 -> 0.00 mm, vias 6 -> 0
- net /GND1: track 11.8 -> 0.00 mm, vias 6 -> 0
- net /GND3: track 11.6 -> 0.00 mm, vias 6 -> 0
- net /GND2: track 11.4 -> 0.00 mm, vias 6 -> 0
- net 5V: track 49.7 -> 59.8 mm, vias 24 -> 28
- net Net-(D1-A): track 0.00 -> 7.98 mm
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- added copper zone on In1.Cu, net GND1
- added copper zone on In1.Cu, net GND2
- added copper zone on In1.Cu, net GND3
- added copper zone on In1.Cu, net GND4
- removed copper zone on In1.Cu, net /GND1
- removed copper zone on In1.Cu, net /GND2
- removed copper zone on In1.Cu, net /GND3
- removed copper zone on In1.Cu, net /GND4
Other:
- board size 129.8 x 129 mm -> 131 x 129 mm
- board text added: "DISK 1"
- board text added: "DISK 2"
- board text added: "DISK 3"
- board text added: "DISK 4"
- board text added: "SATA 1"
- board text added: "SATA 2"
- board text added: "SATA 3"
- board text added: "SATA 4"
- board text removed: "HDD_1"
- board text removed: "HDD_2"
- board text removed: "HDD_3"
- board text removed: "HDD_4"
- board text removed: "SATA_1"
- board text removed: "SATA_2"
- board text removed: "SATA_3"
- board text removed: "SATA_4"
