File: 8x-sata-backplane/8x-sata-backplane.kicad_sch (KiCad schematic)
At the start: 9 parts

Commit message: v1.0
Parts:
- added D1, D2, D3, D4: LED, LED_SMD:LED_0603_1608Metric, symbol Device:LED
- added Q1, Q2, Q3, Q4: BC850, Package_TO_SOT_SMD:SOT-23, symbol Transistor_BJT:BC850
- added R1, R10, R12, R3, R4, R6, R7, R9: 1k, Resistor_SMD:R_0805_2012Metric, symbol Device:R
- added R11, R2, R5, R8: 330, Resistor_SMD:R_0805_2012Metric, symbol Device:R
- J1, J3, J5, J7: footprint shirnschall:SATA BACKPLANE RECPT VERTICAL SMT -> shirnschall:sata-backplane-connector-vert
Connections:
- net 5V: now also R1.1, R10.1, R11.2, R2.2, R4.1, R5.2, R7.1, R8.2
- net GND: now also R12.2, R3.2, R6.2, R9.2; no longer J1.18 (P11), J3.18 (P11), J5.18 (P11), J7.18 (P11)
- net GND1: now also J1.23 (C1), J2.8 (C1), J2.9 (C2)
- net GND2: now also J3.23 (C1), J4.8 (C1), J4.9 (C2)
- net GND3: now also J5.23 (C1), J6.8 (C1), J6.9 (C2)
- net GND4: now also J7.23 (C1), J8.8 (C1), J8.9 (C2)
- new net: D1.1 (K), Q1.2 (E), R3.1
- new net: D1.2 (A), Q1.3 (C), R2.1
- new net: D3.1 (K), Q3.2 (E), R9.1
- new net: D2.1 (K), Q2.2 (E), R6.1
- new net: D4.1 (K), Q4.2 (E), R12.1
- new net: D2.2 (A), Q2.3 (C), R5.1
- new net: D3.2 (A), Q3.3 (C), R8.1
- new net: D4.2 (A), Q4.3 (C), R11.1
- new net 1_ACT: J1.18 (P11), Q1.1 (B), R1.2
- new net 2_ACT: J3.18 (P11), Q2.1 (B), R4.2
- new net 3_ACT: J5.18 (P11), Q3.1 (B), R7.2
- new net 4_ACT: J7.18 (P11), Q4.1 (B), R10.2
- no-connect marks 28 -> 16
Other:
- note added: "DRIVE ACTIVITY"
